File: Production/12359_HiBeam_3x3.kicad_pcb_panel.v10.kicad_pcb (KiCad board)
At the start: 2 copper layers, 185.7 x 105.4 mm, 503 parts, among them J1 Input, J2 Output, U1 APA102, U2 APA102, U3 APA102, U4 APA102, U5 APA102, U6 APA102, U7 APA102, U8 APA102, U9 APA102

Commit message: Protopanelupdate
Parts:
- removed the ? at (161.3, 91.2)
- removed the ? at (23.2, 68.1)
- removed the ? at (161.3, 45.0)
- removed the ? at (126.8, 45.0)
- removed the ? at (92.2, 45.0)
- removed the ? at (57.7, 45.0)
- removed the ? at (23.2, 45.0)
- removed the ? at (161.3, 21.9)
- removed the ? at (126.8, 21.9)
- removed the ? at (92.2, 21.9)
- removed the ? at (57.7, 21.9)
- removed the ? at (126.8, 91.2)
- removed the ? at (23.2, 21.9)
- removed the ? at (92.2, 91.2)
- removed the ? at (57.7, 91.2)
- removed the ? at (23.2, 91.2)
- removed the ? at (161.3, 68.1)
- removed the ? at (126.8, 68.1)
- removed the ? at (92.2, 68.1)
- removed the ? at (57.7, 68.1)
- removed the C1 at (154.3, 97.2)
- removed the C1 at (16.1, 74.1)
- removed the C1 at (154.3, 51.0)
- removed the C1 at (119.8, 51.0)
- removed the C1 at (85.2, 51.0)
- removed the C1 at (50.7, 51.0)
- removed the C1 at (16.1, 51.0)
- removed the C1 at (154.3, 27.9)
- removed the C1 at (119.8, 27.9)
- removed the C1 at (85.2, 27.9)
- removed the C1 at (50.7, 27.9)
- removed the C1 at (119.8, 97.2)
- removed the C1 at (16.1, 27.9)
- removed the C1 at (85.2, 97.2)
- removed the C1 at (50.7, 97.2)
- removed the C1 at (16.1, 97.2)
- removed the C1 at (154.3, 74.1)
- removed the C1 at (119.8, 74.1)
- removed the C1 at (85.2, 74.1)
- removed the C1 at (50.7, 74.1)
- removed the C2 at (127.4, 97.2)
- removed the C2 at (23.8, 74.1)
- removed the C2 at (127.4, 51.0)
- removed the C2 at (162.0, 51.0)
- removed the C2 at (92.9, 51.0)
- removed the C2 at (58.3, 51.0)
- removed the C2 at (23.8, 51.0)
- removed the C2 at (162.0, 27.9)
- removed the C2 at (127.4, 27.9)
- removed the C2 at (92.9, 27.9)
- removed the C2 at (58.3, 27.9)
- removed the C2 at (162.0, 97.2)
- removed the C2 at (23.8, 27.9)
- removed the C2 at (92.9, 97.2)
- removed the C2 at (58.3, 97.2)
- removed the C2 at (23.8, 97.2)
- removed the C2 at (127.4, 74.1)
- removed the C2 at (162.0, 74.1)
- removed the C2 at (92.9, 74.1)
- removed the C2 at (58.3, 74.1)
- removed the C3 at (169.5, 97.2)
- removed the C3 at (31.4, 74.1)
- removed the C3 at (169.5, 51.0)
- removed the C3 at (135.0, 51.0)
- removed the C3 at (100.5, 51.0)
- removed the C3 at (65.9, 51.0)
- removed the C3 at (31.4, 51.0)
- removed the C3 at (169.5, 27.9)
- removed the C3 at (135.0, 27.9)
- removed the C3 at (100.5, 27.9)
- removed the C3 at (65.9, 27.9)
- removed the C3 at (135.0, 97.2)
- removed the C3 at (31.4, 27.9)
- removed the C3 at (100.5, 97.2)
- removed the C3 at (65.9, 97.2)
- removed the C3 at (31.4, 97.2)
- removed the C3 at (169.5, 74.1)
- removed the C3 at (135.0, 74.1)
- removed the C3 at (100.5, 74.1)
- removed the C3 at (65.9, 74.1)
- removed the C4 at (135.0, 83.2)
- removed the C4 at (31.4, 60.1)
- removed the C4 at (135.0, 37.0)
- removed the C4 at (169.5, 37.0)
- removed the C4 at (100.5, 37.0)
- removed the C4 at (65.9, 37.0)
- removed the C4 at (31.4, 37.0)
- removed the C4 at (169.5, 13.9)
- removed the C4 at (135.0, 13.9)
- removed the C4 at (100.5, 13.9)
- removed the C4 at (65.9, 13.9)
- removed the C4 at (169.5, 83.2)
- removed the C4 at (31.4, 13.9)
- removed the C4 at (100.5, 83.2)
- removed the C4 at (65.9, 83.2)
- removed the C4 at (31.4, 83.2)
- removed the C4 at (135.0, 60.1)
- removed the C4 at (169.5, 60.1)
- removed the C4 at (100.5, 60.1)
- removed the C4 at (65.9, 60.1)
- removed the C5 at (162.0, 83.3)
- removed the C5 at (23.8, 60.1)
- removed the C5 at (162.0, 37.0)
- removed the C5 at (127.4, 37.0)
- removed the C5 at (92.9, 37.0)
- removed the C5 at (58.3, 37.0)
- removed the C5 at (23.8, 37.0)
- removed the C5 at (162.0, 13.9)
- removed the C5 at (127.4, 13.9)
- removed the C5 at (92.9, 13.9)
- removed the C5 at (58.3, 13.9)
- removed the C5 at (127.4, 83.3)
- removed the C5 at (23.8, 13.9)
- removed the C5 at (92.9, 83.3)
- removed the C5 at (58.3, 83.3)
- removed the C5 at (23.8, 83.3)
- removed the C5 at (162.0, 60.1)
- removed the C5 at (127.4, 60.1)
- removed the C5 at (92.9, 60.1)
- removed the C5 at (58.3, 60.1)
- removed the C6 at (154.3, 83.3)
- removed the C6 at (16.1, 60.1)
- removed the C6 at (154.3, 37.0)
- removed the C6 at (119.8, 37.0)
- removed the C6 at (85.2, 37.0)
- removed the C6 at (50.7, 37.0)
- removed the C6 at (16.1, 37.0)
- removed the C6 at (154.3, 13.9)
- removed the C6 at (119.8, 13.9)
- removed the C6 at (85.2, 13.9)
- removed the C6 at (50.7, 13.9)
- removed the C6 at (119.8, 83.3)
- removed the C6 at (16.1, 13.9)
- removed the C6 at (85.2, 83.3)
- removed the C6 at (50.7, 83.3)
- removed the C6 at (16.1, 83.3)
- removed the C6 at (154.3, 60.1)
- removed the C6 at (119.8, 60.1)
- removed the C6 at (85.2, 60.1)
- removed the C6 at (50.7, 60.1)
- removed the FD1 at (143.3, 77.2)
- removed the FD1 at (39.6, 54.1)
- removed the FD1 at (143.3, 31.0)
- removed the FD1 at (177.8, 31.0)
- removed the FD1 at (108.7, 31.0)
- removed the FD1 at (74.2, 31.0)
- removed the FD1 at (39.6, 31.0)
- removed the FD1 at (177.8, 7.87)
- removed the FD1 at (143.3, 7.87)
- removed the FD1 at (108.7, 7.87)
- removed the FD1 at (74.2, 7.87)
- removed the FD1 at (177.8, 77.2)
- removed the FD1 at (39.6, 7.87)
- removed the FD1 at (108.7, 77.2)
- removed the FD1 at (74.2, 77.2)
- removed the FD1 at (39.6, 77.2)
- removed the FD1 at (143.3, 54.1)
- removed the FD1 at (177.8, 54.1)
- removed the FD1 at (108.7, 54.1)
- removed the FD1 at (74.2, 54.1)
- removed the FD2 at (146.1, 97.5)
- removed the FD2 at (42.4, 74.4)
- removed the FD2 at (146.1, 51.3)
- removed the FD2 at (111.5, 51.3)
- removed the FD2 at (77.0, 51.3)
- removed the FD2 at (7.87, 51.3)
- removed the FD2 at (42.4, 51.3)
- removed the FD2 at (146.1, 28.2)
- removed the FD2 at (111.5, 28.2)
- removed the FD2 at (77.0, 28.2)
- removed the FD2 at (42.4, 28.2)
- removed the FD2 at (111.5, 97.5)
- removed the FD2 at (7.87, 28.2)
- removed the FD2 at (77.0, 97.5)
- removed the FD2 at (7.87, 97.5)
- removed the FD2 at (42.4, 97.5)
- removed the FD2 at (146.1, 74.4)
- removed the FD2 at (111.5, 74.4)
- removed the FD2 at (77.0, 74.4)
- removed the FD2 at (7.87, 74.4)
- removed the J1 at (146.1, 83.6)
- removed the J1 at (42.4, 60.5)
- removed the J1 at (146.1, 37.3)
- removed the J1 at (111.5, 37.3)
- removed the J1 at (77.0, 37.3)
- removed the J1 at (7.87, 37.3)
- removed the J1 at (42.4, 37.3)
- removed the J1 at (146.1, 14.2)
- removed the J1 at (111.5, 14.2)
- removed the J1 at (77.0, 14.2)
- removed the J1 at (42.4, 14.2)
- removed the J1 at (111.5, 83.6)
- removed the J1 at (7.87, 14.2)
- removed the J1 at (77.0, 83.6)
- removed the J1 at (7.87, 83.6)
- removed the J1 at (42.4, 83.6)
- removed the J1 at (146.1, 60.5)
- removed the J1 at (111.5, 60.5)
- removed the J1 at (77.0, 60.5)
- removed the J1 at (7.87, 60.5)
- removed the J2 at (143.3, 91.2)
- removed the J2 at (39.6, 68.1)
- removed the J2 at (143.3, 45.0)
- removed the J2 at (177.8, 45.0)
- removed the J2 at (108.7, 45.0)
- removed the J2 at (74.2, 45.0)
- removed the J2 at (39.6, 45.0)
- removed the J2 at (177.8, 21.8)
- removed the J2 at (143.3, 21.8)
- removed the J2 at (108.7, 21.8)
- removed the J2 at (74.2, 21.8)
- removed the J2 at (177.8, 91.2)
- removed the J2 at (39.6, 21.8)
- removed the J2 at (108.7, 91.2)
- removed the J2 at (74.2, 91.2)
- removed the J2 at (39.6, 91.2)
- removed the J2 at (143.3, 68.1)
- removed the J2 at (177.8, 68.1)
- removed the J2 at (108.7, 68.1)
- removed the J2 at (74.2, 68.1)
- removed the LOGO1 at (167.3, 86.5)
- removed the LOGO1 at (29.1, 63.4)
- removed the LOGO1 at (167.3, 40.3)
- removed the LOGO1 at (98.2, 40.3)
- removed the LOGO1 at (132.7, 40.3)
- removed the LOGO1 at (63.6, 40.3)
- removed the LOGO1 at (29.1, 40.3)
- removed the LOGO1 at (167.3, 17.1)
- removed the LOGO1 at (132.7, 17.1)
- removed the LOGO1 at (98.2, 17.1)
- removed the LOGO1 at (63.6, 17.1)
- removed the LOGO1 at (98.2, 86.5)
- removed the LOGO1 at (29.1, 17.1)
- removed the LOGO1 at (132.7, 86.5)
- removed the LOGO1 at (63.6, 86.5)
- removed the LOGO1 at (29.1, 86.5)
- removed the LOGO1 at (167.3, 63.4)
- removed the LOGO1 at (98.2, 63.4)
- removed the LOGO1 at (132.7, 63.4)
- removed the LOGO1 at (63.6, 63.4)
- removed the LOGO2 at (147.7, 94.9)
- removed the LOGO2 at (44.1, 71.8)
- removed the LOGO2 at (147.7, 48.7)
- removed the LOGO2 at (113.2, 48.7)
- removed the LOGO2 at (78.6, 48.7)
- removed the LOGO2 at (9.53, 48.7)
- removed the LOGO2 at (44.1, 48.7)
- removed the LOGO2 at (147.7, 25.6)
- removed the LOGO2 at (113.2, 25.6)
- removed the LOGO2 at (78.6, 25.6)
- removed the LOGO2 at (44.1, 25.6)
- removed the LOGO2 at (113.2, 94.9)
- removed the LOGO2 at (9.53, 25.6)
- removed the LOGO2 at (78.6, 94.9)
- removed the LOGO2 at (9.53, 94.9)
- removed the LOGO2 at (44.1, 94.9)
- removed the LOGO2 at (147.7, 71.8)
- removed the LOGO2 at (113.2, 71.8)
- removed the LOGO2 at (78.6, 71.8)
- removed the LOGO2 at (9.53, 71.8)
- removed the LOGO3 at (139.3, 82.5)
- removed the LOGO3 at (35.7, 59.4)
- removed the LOGO3 at (139.3, 36.3)
- removed the LOGO3 at (173.9, 36.3)
- removed the LOGO3 at (104.8, 36.3)
- removed the LOGO3 at (70.3, 36.3)
- removed the LOGO3 at (35.7, 36.3)
- removed the LOGO3 at (173.9, 13.2)
- removed the LOGO3 at (139.3, 13.2)
- removed the LOGO3 at (104.8, 13.2)
- removed the LOGO3 at (70.3, 13.2)
- removed the LOGO3 at (173.9, 82.5)
- removed the LOGO3 at (35.7, 13.2)
- removed the LOGO3 at (104.8, 82.5)
- removed the LOGO3 at (70.3, 82.5)
- removed the LOGO3 at (35.7, 82.5)
- removed the LOGO3 at (139.3, 59.4)
- removed the LOGO3 at (173.9, 59.4)
- removed the LOGO3 at (104.8, 59.4)
- removed the LOGO3 at (70.3, 59.4)
- removed the Ref** at (147.6, 78.7)
- removed the Ref** at (38.1, 96.0)
- removed the Ref** at (147.6, 55.6)
- removed the Ref** at (141.7, 72.9)
- removed the Ref** at (176.3, 72.9)
- removed the Ref** at (113.0, 55.6)
- removed the Ref** at (107.2, 72.9)
- removed the Ref** at (78.5, 55.6)
- removed the Ref** at (72.6, 72.9)
- removed the Ref** at (43.9, 55.6)
- removed the Ref** at (9.40, 55.6)
- removed the Ref** at (141.7, 96.0)
- removed the Ref** at (38.1, 72.9)
- removed the Ref** at (147.6, 32.5)
- removed the Ref** at (141.7, 49.8)
- removed the Ref** at (176.3, 49.8)
- removed the Ref** at (113.0, 32.5)
- removed the Ref** at (107.2, 49.8)
- removed the Ref** at (78.5, 32.5)
- removed the Ref** at (72.6, 49.8)
- removed the Ref** at (43.9, 32.5)
- removed the Ref** at (9.40, 32.5)
- removed the Ref** at (176.3, 96.0)
- removed the Ref** at (38.1, 49.8)
- removed the Ref** at (147.6, 9.40)
- removed the Ref** at (176.3, 26.7)
- removed the Ref** at (113.0, 9.40)
- removed the Ref** at (141.7, 26.7)
- removed the Ref** at (78.5, 9.40)
- removed the Ref** at (107.2, 26.7)
- removed the Ref** at (43.9, 9.40)
- removed the Ref** at (72.6, 26.7)
- removed the Ref** at (9.40, 9.40)
- removed the Ref** at (113.0, 78.7)
- removed the Ref** at (38.1, 26.7)
- removed the Ref** at (107.2, 96.0)
- removed the Ref** at (78.5, 78.7)
- removed the Ref** at (72.6, 96.0)
- removed the Ref** at (43.9, 78.7)
- removed the Ref** at (9.40, 78.7)
- removed the U1 at (154.3, 93.7)
- removed the U1 at (16.1, 70.6)
- removed the U1 at (154.3, 47.5)
- removed the U1 at (119.8, 47.5)
- removed the U1 at (85.2, 47.5)
- removed the U1 at (50.7, 47.5)
- removed the U1 at (16.1, 47.5)
- removed the U1 at (154.3, 24.4)
- removed the U1 at (119.8, 24.4)
- removed the U1 at (85.2, 24.4)
- removed the U1 at (50.7, 24.4)
- removed the U1 at (119.8, 93.7)
- removed the U1 at (16.1, 24.4)
- removed the U1 at (85.2, 93.7)
- removed the U1 at (50.7, 93.7)
- removed the U1 at (16.1, 93.7)
- removed the U1 at (154.3, 70.6)
- removed the U1 at (119.8, 70.6)
- removed the U1 at (85.2, 70.6)
- removed the U1 at (50.7, 70.6)
- removed the U2 at (127.4, 93.7)
- removed the U2 at (23.7, 70.6)
- removed the U2 at (127.4, 47.5)
- removed the U2 at (161.9, 47.5)
- removed the U2 at (92.8, 47.5)
- removed the U2 at (58.3, 47.5)
- removed the U2 at (23.7, 47.5)
- removed the U2 at (161.9, 24.4)
- removed the U2 at (127.4, 24.4)
- removed the U2 at (92.8, 24.4)
- removed the U2 at (58.3, 24.4)
- removed the U2 at (161.9, 93.7)
- removed the U2 at (23.7, 24.4)
- removed the U2 at (92.8, 93.7)
- removed the U2 at (58.3, 93.7)
- removed the U2 at (23.7, 93.7)
- removed the U2 at (127.4, 70.6)
- removed the U2 at (161.9, 70.6)
- removed the U2 at (92.8, 70.6)
- removed the U2 at (58.3, 70.6)
- removed the U3 at (135.0, 93.7)
- removed the U3 at (31.4, 70.6)
- removed the U3 at (135.0, 47.5)
- removed the U3 at (169.5, 47.5)
- removed the U3 at (100.5, 47.5)
- removed the U3 at (65.9, 47.5)
- removed the U3 at (31.4, 47.5)
- removed the U3 at (169.5, 24.4)
- removed the U3 at (135.0, 24.4)
- removed the U3 at (100.5, 24.4)
- removed the U3 at (65.9, 24.4)
- removed the U3 at (169.5, 93.7)
- removed the U3 at (31.4, 24.4)
- removed the U3 at (100.5, 93.7)
- removed the U3 at (65.9, 93.7)
- removed the U3 at (31.4, 93.7)
- removed the U3 at (135.0, 70.6)
- removed the U3 at (169.5, 70.6)
- removed the U3 at (100.5, 70.6)
- removed the U3 at (65.9, 70.6)
- removed the U4 at (135.0, 86.7)
- removed the U4 at (31.4, 63.6)
- removed the U4 at (135.0, 40.5)
- removed the U4 at (169.5, 40.5)
- removed the U4 at (100.5, 40.5)
- removed the U4 at (65.9, 40.5)
- removed the U4 at (31.4, 40.5)
- removed the U4 at (169.5, 17.4)
- removed the U4 at (135.0, 17.4)
- removed the U4 at (100.5, 17.4)
- removed the U4 at (65.9, 17.4)
- removed the U4 at (169.5, 86.7)
- removed the U4 at (31.4, 17.4)
- removed the U4 at (100.5, 86.7)
- removed the U4 at (65.9, 86.7)
- removed the U4 at (31.4, 86.7)
- removed the U4 at (135.0, 63.6)
- removed the U4 at (169.5, 63.6)
- removed the U4 at (100.5, 63.6)
- removed the U4 at (65.9, 63.6)
- removed the U5 at (161.9, 86.7)
- removed the U5 at (23.7, 63.6)
- removed the U5 at (161.9, 40.5)
- removed the U5 at (127.4, 40.5)
- removed the U5 at (92.8, 40.5)
- removed the U5 at (58.3, 40.5)
- removed the U5 at (23.7, 40.5)
- removed the U5 at (161.9, 17.4)
- removed the U5 at (127.4, 17.4)
- removed the U5 at (92.8, 17.4)
- removed the U5 at (58.3, 17.4)
- removed the U5 at (127.4, 86.7)
- removed the U5 at (23.7, 17.4)
- removed the U5 at (92.8, 86.7)
- removed the U5 at (58.3, 86.7)
- removed the U5 at (23.7, 86.7)
- removed the U5 at (161.9, 63.6)
- removed the U5 at (127.4, 63.6)
- removed the U5 at (92.8, 63.6)
- removed the U5 at (58.3, 63.6)
- removed the U6 at (154.3, 86.7)
- removed the U6 at (16.1, 63.6)
- removed the U6 at (154.3, 40.5)
- removed the U6 at (119.8, 40.5)
- removed the U6 at (85.2, 40.5)
- removed the U6 at (50.7, 40.5)
- removed the U6 at (16.1, 40.5)
- removed the U6 at (154.3, 17.4)
- removed the U6 at (119.8, 17.4)
- removed the U6 at (85.2, 17.4)
- removed the U6 at (50.7, 17.4)
- removed the U6 at (119.8, 86.7)
- removed the U6 at (16.1, 17.4)
- removed the U6 at (85.2, 86.7)
- removed the U6 at (50.7, 86.7)
- removed the U6 at (16.1, 86.7)
- removed the U6 at (154.3, 63.6)
- removed the U6 at (119.8, 63.6)
- removed the U6 at (85.2, 63.6)
- removed the U6 at (50.7, 63.6)
- removed the U7 at (154.3, 79.8)
- removed the U7 at (16.1, 56.6)
- removed the U7 at (154.3, 33.5)
- removed the U7 at (119.8, 33.5)
- removed the U7 at (85.2, 33.5)
- removed the U7 at (50.7, 33.5)
- removed the U7 at (16.1, 33.5)
- removed the U7 at (154.3, 10.4)
- removed the U7 at (119.8, 10.4)
- removed the U7 at (85.2, 10.4)
- removed the U7 at (50.7, 10.4)
- removed the U7 at (119.8, 79.8)
- removed the U7 at (16.1, 10.4)
- removed the U7 at (85.2, 79.8)
- removed the U7 at (50.7, 79.8)
- removed the U7 at (16.1, 79.8)
- removed the U7 at (154.3, 56.6)
- removed the U7 at (119.8, 56.6)
- removed the U7 at (85.2, 56.6)
- removed the U7 at (50.7, 56.6)
- removed the U8 at (127.4, 79.8)
- removed the U8 at (23.7, 56.6)
- removed the U8 at (127.4, 33.5)
- removed the U8 at (161.9, 33.5)
- removed the U8 at (92.8, 33.5)
- removed the U8 at (58.3, 33.5)
- removed the U8 at (23.7, 33.5)
- removed the U8 at (161.9, 10.4)
- removed the U8 at (127.4, 10.4)
- removed the U8 at (92.8, 10.4)
- removed the U8 at (58.3, 10.4)
- removed the U8 at (161.9, 79.8)
- removed the U8 at (23.7, 10.4)
- removed the U8 at (92.8, 79.8)
- removed the U8 at (58.3, 79.8)
- removed the U8 at (23.7, 79.8)
- removed the U8 at (127.4, 56.6)
- removed the U8 at (161.9, 56.6)
- removed the U8 at (92.8, 56.6)
- removed the U8 at (58.3, 56.6)
- removed the U9 at (135.0, 79.8)
- removed the U9 at (31.4, 56.6)
- removed the U9 at (135.0, 33.5)
- removed the U9 at (169.5, 33.5)
- removed the U9 at (100.5, 33.5)
- removed the U9 at (65.9, 33.5)
- removed the U9 at (31.4, 33.5)
- removed the U9 at (169.5, 10.4)
- removed the U9 at (135.0, 10.4)
- removed the U9 at (100.5, 10.4)
- removed the U9 at (65.9, 10.4)
- removed the U9 at (169.5, 79.8)
- removed the U9 at (31.4, 10.4)
- removed the U9 at (100.5, 79.8)
- removed the U9 at (65.9, 79.8)
- removed the U9 at (31.4, 79.8)
- removed the U9 at (135.0, 56.6)
- removed the U9 at (169.5, 56.6)
- removed the U9 at (100.5, 56.6)
- removed the U9 at (65.9, 56.6)
- added ?: , Aesthetics:OSHW-LOGO-M, B.Cu at (218.6, 138.0)
- added ?: , Aesthetics:OSHW-LOGO-M, B.Cu at (80.4, 114.9)
- added ?: , Aesthetics:OSHW-LOGO-M, B.Cu at (218.6, 91.7)
- added ?: , Aesthetics:OSHW-LOGO-M, B.Cu at (184.1, 91.7)
- added ?: , Aesthetics:OSHW-LOGO-M, B.Cu at (149.5, 91.7)
- added ?: , Aesthetics:OSHW-LOGO-M, B.Cu at (115.0, 91.7)
- added ?: , Aesthetics:OSHW-LOGO-M, B.Cu at (80.4, 91.7)
- added ?: , Aesthetics:OSHW-LOGO-M, B.Cu at (218.6, 68.6)
- added ?: , Aesthetics:OSHW-LOGO-M, B.Cu at (184.1, 68.6)
- added ?: , Aesthetics:OSHW-LOGO-M, B.Cu at (149.5, 68.6)
- added ?: , Aesthetics:OSHW-LOGO-M, B.Cu at (115.0, 68.6)
- added ?: , Aesthetics:OSHW-LOGO-M, B.Cu at (184.1, 138.0)
- added ?: , Aesthetics:OSHW-LOGO-M, B.Cu at (80.4, 68.6)
- added ?: , Aesthetics:OSHW-LOGO-M, B.Cu at (149.5, 138.0)
- added ?: , Aesthetics:OSHW-LOGO-M, B.Cu at (115.0, 138.0)
- added ?: , Aesthetics:OSHW-LOGO-M, B.Cu at (80.4, 138.0)
- added ?: , Aesthetics:OSHW-LOGO-M, B.Cu at (218.6, 114.9)
- added ?: , Aesthetics:OSHW-LOGO-M, B.Cu at (184.1, 114.9)
- added ?: , Aesthetics:OSHW-LOGO-M, B.Cu at (149.5, 114.9)
- added ?: , Aesthetics:OSHW-LOGO-M, B.Cu at (115.0, 114.9)
- added C1: 0.1uF, Pete:0603_revised, F.Cu at (211.6, 143.9)
- added C1: 0.1uF, Pete:0603_revised, F.Cu at (73.4, 120.8)
- added C1: 0.1uF, Pete:0603_revised, F.Cu at (211.6, 97.7)
- added C1: 0.1uF, Pete:0603_revised, F.Cu at (142.5, 97.7)
- added C1: 0.1uF, Pete:0603_revised, F.Cu at (108.0, 97.7)
- added C1: 0.1uF, Pete:0603_revised, F.Cu at (177.0, 97.7)
- added C1: 0.1uF, Pete:0603_revised, F.Cu at (73.4, 97.7)
- added C1: 0.1uF, Pete:0603_revised, F.Cu at (211.6, 74.6)
- added C1: 0.1uF, Pete:0603_revised, F.Cu at (177.0, 74.6)
- added C1: 0.1uF, Pete:0603_revised, F.Cu at (142.5, 74.6)
- added C1: 0.1uF, Pete:0603_revised, F.Cu at (108.0, 74.6)
- added C1: 0.1uF, Pete:0603_revised, F.Cu at (142.5, 143.9)
- added C1: 0.1uF, Pete:0603_revised, F.Cu at (73.4, 74.6)
- added C1: 0.1uF, Pete:0603_revised, F.Cu at (108.0, 143.9)
- added C1: 0.1uF, Pete:0603_revised, F.Cu at (177.0, 143.9)
- added C1: 0.1uF, Pete:0603_revised, F.Cu at (73.4, 143.9)
- added C1: 0.1uF, Pete:0603_revised, F.Cu at (211.6, 120.8)
- added C1: 0.1uF, Pete:0603_revised, F.Cu at (142.5, 120.8)
- added C1: 0.1uF, Pete:0603_revised, F.Cu at (108.0, 120.8)
- added C1: 0.1uF, Pete:0603_revised, F.Cu at (177.0, 120.8)
- added C2: 0.1uF, Pete:0603_revised, F.Cu at (219.2, 143.9)
- added C2: 0.1uF, Pete:0603_revised, F.Cu at (81.1, 120.8)
- added C2: 0.1uF, Pete:0603_revised, F.Cu at (219.2, 97.7)
- added C2: 0.1uF, Pete:0603_revised, F.Cu at (150.1, 97.7)
- added C2: 0.1uF, Pete:0603_revised, F.Cu at (115.6, 97.7)
- added C2: 0.1uF, Pete:0603_revised, F.Cu at (184.7, 97.7)
- added C2: 0.1uF, Pete:0603_revised, F.Cu at (81.1, 97.7)
- added C2: 0.1uF, Pete:0603_revised, F.Cu at (219.2, 74.6)
- added C2: 0.1uF, Pete:0603_revised, F.Cu at (184.7, 74.6)
- added C2: 0.1uF, Pete:0603_revised, F.Cu at (150.1, 74.6)
- added C2: 0.1uF, Pete:0603_revised, F.Cu at (115.6, 74.6)
- added C2: 0.1uF, Pete:0603_revised, F.Cu at (150.1, 143.9)
- added C2: 0.1uF, Pete:0603_revised, F.Cu at (81.1, 74.6)
- added C2: 0.1uF, Pete:0603_revised, F.Cu at (115.6, 143.9)
- added C2: 0.1uF, Pete:0603_revised, F.Cu at (184.7, 143.9)
- added C2: 0.1uF, Pete:0603_revised, F.Cu at (81.1, 143.9)
- added C2: 0.1uF, Pete:0603_revised, F.Cu at (219.2, 120.8)
- added C2: 0.1uF, Pete:0603_revised, F.Cu at (150.1, 120.8)
- added C2: 0.1uF, Pete:0603_revised, F.Cu at (115.6, 120.8)
- added C2: 0.1uF, Pete:0603_revised, F.Cu at (184.7, 120.8)
- added C3: 0.1uF, Pete:0603_revised, F.Cu at (226.8, 143.9)
- added C3: 0.1uF, Pete:0603_revised, F.Cu at (88.6, 120.8)
- added C3: 0.1uF, Pete:0603_revised, F.Cu at (226.8, 97.7)
- added C3: 0.1uF, Pete:0603_revised, F.Cu at (157.7, 97.7)
- added C3: 0.1uF, Pete:0603_revised, F.Cu at (123.2, 97.7)
- added C3: 0.1uF, Pete:0603_revised, F.Cu at (192.3, 97.7)
- added C3: 0.1uF, Pete:0603_revised, F.Cu at (88.6, 97.7)
- added C3: 0.1uF, Pete:0603_revised, F.Cu at (226.8, 74.6)
- added C3: 0.1uF, Pete:0603_revised, F.Cu at (192.3, 74.6)
- added C3: 0.1uF, Pete:0603_revised, F.Cu at (157.7, 74.6)
- added C3: 0.1uF, Pete:0603_revised, F.Cu at (123.2, 74.6)
- added C3: 0.1uF, Pete:0603_revised, F.Cu at (157.7, 143.9)
- added C3: 0.1uF, Pete:0603_revised, F.Cu at (88.6, 74.6)
- added C3: 0.1uF, Pete:0603_revised, F.Cu at (123.2, 143.9)
- added C3: 0.1uF, Pete:0603_revised, F.Cu at (192.3, 143.9)
- added C3: 0.1uF, Pete:0603_revised, F.Cu at (88.6, 143.9)
- added C3: 0.1uF, Pete:0603_revised, F.Cu at (226.8, 120.8)
- added C3: 0.1uF, Pete:0603_revised, F.Cu at (157.7, 120.8)
- added C3: 0.1uF, Pete:0603_revised, F.Cu at (123.2, 120.8)
- added C3: 0.1uF, Pete:0603_revised, F.Cu at (192.3, 120.8)
- added C4: 0.22uF, Pete:0603_revised, F.Cu at (226.8, 130.0)
- added C4: 0.22uF, Pete:0603_revised, F.Cu at (192.3, 106.9)
- added C4: 0.22uF, Pete:0603_revised, F.Cu at (226.8, 83.7)
- added C4: 0.22uF, Pete:0603_revised, F.Cu at (157.7, 83.7)
- added C4: 0.22uF, Pete:0603_revised, F.Cu at (123.2, 83.7)
- added C4: 0.22uF, Pete:0603_revised, F.Cu at (88.6, 83.7)
- added C4: 0.22uF, Pete:0603_revised, F.Cu at (192.3, 83.7)
- added C4: 0.22uF, Pete:0603_revised, F.Cu at (226.8, 60.6)
- added C4: 0.22uF, Pete:0603_revised, F.Cu at (192.3, 60.6)
- added C4: 0.22uF, Pete:0603_revised, F.Cu at (157.7, 60.6)
- added C4: 0.22uF, Pete:0603_revised, F.Cu at (123.2, 60.6)
- added C4: 0.22uF, Pete:0603_revised, F.Cu at (157.7, 130.0)
- added C4: 0.22uF, Pete:0603_revised, F.Cu at (88.6, 60.6)
- added C4: 0.22uF, Pete:0603_revised, F.Cu at (123.2, 130.0)
- added C4: 0.22uF, Pete:0603_revised, F.Cu at (88.6, 130.0)
- added C4: 0.22uF, Pete:0603_revised, F.Cu at (192.3, 130.0)
- added C4: 0.22uF, Pete:0603_revised, F.Cu at (226.8, 106.9)
- added C4: 0.22uF, Pete:0603_revised, F.Cu at (157.7, 106.9)
- added C4: 0.22uF, Pete:0603_revised, F.Cu at (123.2, 106.9)
- added C4: 0.22uF, Pete:0603_revised, F.Cu at (88.6, 106.9)
- added C5: 0.22uF, Pete:0603_revised, F.Cu at (219.2, 130.0)
- added C5: 0.22uF, Pete:0603_revised, F.Cu at (81.1, 106.9)
- added C5: 0.22uF, Pete:0603_revised, F.Cu at (219.2, 83.8)
- added C5: 0.22uF, Pete:0603_revised, F.Cu at (150.1, 83.8)
- added C5: 0.22uF, Pete:0603_revised, F.Cu at (115.6, 83.8)
- added C5: 0.22uF, Pete:0603_revised, F.Cu at (184.7, 83.8)
- added C5: 0.22uF, Pete:0603_revised, F.Cu at (81.1, 83.8)
- added C5: 0.22uF, Pete:0603_revised, F.Cu at (219.2, 60.7)
- added C5: 0.22uF, Pete:0603_revised, F.Cu at (184.7, 60.7)
- added C5: 0.22uF, Pete:0603_revised, F.Cu at (150.1, 60.7)
- added C5: 0.22uF, Pete:0603_revised, F.Cu at (115.6, 60.7)
- added C5: 0.22uF, Pete:0603_revised, F.Cu at (150.1, 130.0)
- added C5: 0.22uF, Pete:0603_revised, F.Cu at (81.1, 60.7)
- added C5: 0.22uF, Pete:0603_revised, F.Cu at (115.6, 130.0)
- added C5: 0.22uF, Pete:0603_revised, F.Cu at (184.7, 130.0)
- added C5: 0.22uF, Pete:0603_revised, F.Cu at (81.1, 130.0)
- added C5: 0.22uF, Pete:0603_revised, F.Cu at (219.2, 106.9)
- added C5: 0.22uF, Pete:0603_revised, F.Cu at (150.1, 106.9)
- added C5: 0.22uF, Pete:0603_revised, F.Cu at (115.6, 106.9)
- added C5: 0.22uF, Pete:0603_revised, F.Cu at (184.7, 106.9)
- added C6: 0.22uF, Pete:0603_revised, F.Cu at (211.6, 130.0)
- added C6: 0.22uF, Pete:0603_revised, F.Cu at (73.4, 106.9)
- added C6: 0.22uF, Pete:0603_revised, F.Cu at (211.6, 83.8)
- added C6: 0.22uF, Pete:0603_revised, F.Cu at (142.5, 83.8)
- added C6: 0.22uF, Pete:0603_revised, F.Cu at (108.0, 83.8)
- added C6: 0.22uF, Pete:0603_revised, F.Cu at (177.0, 83.8)
- added C6: 0.22uF, Pete:0603_revised, F.Cu at (73.4, 83.8)
- added C6: 0.22uF, Pete:0603_revised, F.Cu at (211.6, 60.7)
- added C6: 0.22uF, Pete:0603_revised, F.Cu at (177.0, 60.7)
- added C6: 0.22uF, Pete:0603_revised, F.Cu at (142.5, 60.7)
- added C6: 0.22uF, Pete:0603_revised, F.Cu at (108.0, 60.7)
- added C6: 0.22uF, Pete:0603_revised, F.Cu at (142.5, 130.0)
- added C6: 0.22uF, Pete:0603_revised, F.Cu at (73.4, 60.7)
- added C6: 0.22uF, Pete:0603_revised, F.Cu at (108.0, 130.0)
- added C6: 0.22uF, Pete:0603_revised, F.Cu at (177.0, 130.0)
- added C6: 0.22uF, Pete:0603_revised, F.Cu at (73.4, 130.0)
- added C6: 0.22uF, Pete:0603_revised, F.Cu at (211.6, 106.9)
- added C6: 0.22uF, Pete:0603_revised, F.Cu at (142.5, 106.9)
- added C6: 0.22uF, Pete:0603_revised, F.Cu at (108.0, 106.9)
- added C6: 0.22uF, Pete:0603_revised, F.Cu at (177.0, 106.9)
- added FD1: FIDUCIAL1X2, Aesthetics:FIDUCIAL-1X2, F.Cu at (235.1, 124.0)
- added FD1: FIDUCIAL1X2, Aesthetics:FIDUCIAL-1X2, F.Cu at (200.5, 100.8)
- added FD1: FIDUCIAL1X2, Aesthetics:FIDUCIAL-1X2, F.Cu at (235.1, 77.7)
- added FD1: FIDUCIAL1X2, Aesthetics:FIDUCIAL-1X2, F.Cu at (166.0, 77.7)
- added FD1: FIDUCIAL1X2, Aesthetics:FIDUCIAL-1X2, F.Cu at (131.4, 77.7)
- added FD1: FIDUCIAL1X2, Aesthetics:FIDUCIAL-1X2, F.Cu at (96.9, 77.7)
- added FD1: FIDUCIAL1X2, Aesthetics:FIDUCIAL-1X2, F.Cu at (200.5, 77.7)
- added FD1: FIDUCIAL1X2, Aesthetics:FIDUCIAL-1X2, F.Cu at (235.1, 54.6)
- added FD1: FIDUCIAL1X2, Aesthetics:FIDUCIAL-1X2, F.Cu at (200.5, 54.6)
- added FD1: FIDUCIAL1X2, Aesthetics:FIDUCIAL-1X2, F.Cu at (166.0, 54.6)
- added FD1: FIDUCIAL1X2, Aesthetics:FIDUCIAL-1X2, F.Cu at (131.4, 54.6)
- added FD1: FIDUCIAL1X2, Aesthetics:FIDUCIAL-1X2, F.Cu at (166.0, 124.0)
- added FD1: FIDUCIAL1X2, Aesthetics:FIDUCIAL-1X2, F.Cu at (96.9, 54.6)
- added FD1: FIDUCIAL1X2, Aesthetics:FIDUCIAL-1X2, F.Cu at (131.4, 124.0)
- added FD1: FIDUCIAL1X2, Aesthetics:FIDUCIAL-1X2, F.Cu at (96.9, 124.0)
- added FD1: FIDUCIAL1X2, Aesthetics:FIDUCIAL-1X2, F.Cu at (200.5, 124.0)
- added FD1: FIDUCIAL1X2, Aesthetics:FIDUCIAL-1X2, F.Cu at (235.1, 100.8)
- added FD1: FIDUCIAL1X2, Aesthetics:FIDUCIAL-1X2, F.Cu at (166.0, 100.8)
- added FD1: FIDUCIAL1X2, Aesthetics:FIDUCIAL-1X2, F.Cu at (131.4, 100.8)
- added FD1: FIDUCIAL1X2, Aesthetics:FIDUCIAL-1X2, F.Cu at (96.9, 100.8)
- added FD2: FIDUCIAL1X2, Aesthetics:FIDUCIAL-1X2, F.Cu at (203.3, 144.3)
- added FD2: FIDUCIAL1X2, Aesthetics:FIDUCIAL-1X2, F.Cu at (65.2, 121.2)
- added FD2: FIDUCIAL1X2, Aesthetics:FIDUCIAL-1X2, F.Cu at (203.3, 98.0)
- added FD2: FIDUCIAL1X2, Aesthetics:FIDUCIAL-1X2, F.Cu at (168.8, 98.0)
- added FD2: FIDUCIAL1X2, Aesthetics:FIDUCIAL-1X2, F.Cu at (134.2, 98.0)
- added FD2: FIDUCIAL1X2, Aesthetics:FIDUCIAL-1X2, F.Cu at (99.7, 98.0)
- added FD2: FIDUCIAL1X2, Aesthetics:FIDUCIAL-1X2, F.Cu at (65.2, 98.0)
- added FD2: FIDUCIAL1X2, Aesthetics:FIDUCIAL-1X2, F.Cu at (203.3, 74.9)
- added FD2: FIDUCIAL1X2, Aesthetics:FIDUCIAL-1X2, F.Cu at (168.8, 74.9)
- added FD2: FIDUCIAL1X2, Aesthetics:FIDUCIAL-1X2, F.Cu at (134.2, 74.9)
- added FD2: FIDUCIAL1X2, Aesthetics:FIDUCIAL-1X2, F.Cu at (99.7, 74.9)
- added FD2: FIDUCIAL1X2, Aesthetics:FIDUCIAL-1X2, F.Cu at (168.8, 144.3)
- added FD2: FIDUCIAL1X2, Aesthetics:FIDUCIAL-1X2, F.Cu at (65.2, 74.9)
- added FD2: FIDUCIAL1X2, Aesthetics:FIDUCIAL-1X2, F.Cu at (134.2, 144.3)
- added FD2: FIDUCIAL1X2, Aesthetics:FIDUCIAL-1X2, F.Cu at (99.7, 144.3)
- added FD2: FIDUCIAL1X2, Aesthetics:FIDUCIAL-1X2, F.Cu at (65.2, 144.3)
- added FD2: FIDUCIAL1X2, Aesthetics:FIDUCIAL-1X2, F.Cu at (203.3, 121.2)
- added FD2: FIDUCIAL1X2, Aesthetics:FIDUCIAL-1X2, F.Cu at (168.8, 121.2)
- added FD2: FIDUCIAL1X2, Aesthetics:FIDUCIAL-1X2, F.Cu at (134.2, 121.2)
- added FD2: FIDUCIAL1X2, Aesthetics:FIDUCIAL-1X2, F.Cu at (99.7, 121.2)
- added J1: Input, SFE_Connectors:1X04_NO_SILK, F.Cu at (203.3, 130.3)
- added J1: Input, SFE_Connectors:1X04_NO_SILK, F.Cu at (65.2, 107.2)
- added J1: Input, SFE_Connectors:1X04_NO_SILK, F.Cu at (203.3, 84.1)
- added J1: Input, SFE_Connectors:1X04_NO_SILK, F.Cu at (168.8, 84.1)
- added J1: Input, SFE_Connectors:1X04_NO_SILK, F.Cu at (134.2, 84.1)
- added J1: Input, SFE_Connectors:1X04_NO_SILK, F.Cu at (99.7, 84.1)
- added J1: Input, SFE_Connectors:1X04_NO_SILK, F.Cu at (65.2, 84.1)
- added J1: Input, SFE_Connectors:1X04_NO_SILK, F.Cu at (203.3, 61.0)
- added J1: Input, SFE_Connectors:1X04_NO_SILK, F.Cu at (168.8, 61.0)
- added J1: Input, SFE_Connectors:1X04_NO_SILK, F.Cu at (134.2, 61.0)
- added J1: Input, SFE_Connectors:1X04_NO_SILK, F.Cu at (99.7, 61.0)
- added J1: Input, SFE_Connectors:1X04_NO_SILK, F.Cu at (168.8, 130.3)
- added J1: Input, SFE_Connectors:1X04_NO_SILK, F.Cu at (65.2, 61.0)
- added J1: Input, SFE_Connectors:1X04_NO_SILK, F.Cu at (134.2, 130.3)
- added J1: Input, SFE_Connectors:1X04_NO_SILK, F.Cu at (99.7, 130.3)
- added J1: Input, SFE_Connectors:1X04_NO_SILK, F.Cu at (65.2, 130.3)
- added J1: Input, SFE_Connectors:1X04_NO_SILK, F.Cu at (203.3, 107.2)
- added J1: Input, SFE_Connectors:1X04_NO_SILK, F.Cu at (168.8, 107.2)
- added J1: Input, SFE_Connectors:1X04_NO_SILK, F.Cu at (134.2, 107.2)
- added J1: Input, SFE_Connectors:1X04_NO_SILK, F.Cu at (99.7, 107.2)
- added J2: Output, SFE_Connectors:1X04_NO_SILK, F.Cu at (235.1, 137.9)
- added J2: Output, SFE_Connectors:1X04_NO_SILK, F.Cu at (200.5, 114.8)
- added J2: Output, SFE_Connectors:1X04_NO_SILK, F.Cu at (235.1, 91.7)
- added J2: Output, SFE_Connectors:1X04_NO_SILK, F.Cu at (166.0, 91.7)
- added J2: Output, SFE_Connectors:1X04_NO_SILK, F.Cu at (131.4, 91.7)
- added J2: Output, SFE_Connectors:1X04_NO_SILK, F.Cu at (96.9, 91.7)
- added J2: Output, SFE_Connectors:1X04_NO_SILK, F.Cu at (200.5, 91.7)
- added J2: Output, SFE_Connectors:1X04_NO_SILK, F.Cu at (235.1, 68.6)
- added J2: Output, SFE_Connectors:1X04_NO_SILK, F.Cu at (200.5, 68.6)
- added J2: Output, SFE_Connectors:1X04_NO_SILK, F.Cu at (166.0, 68.6)
- added J2: Output, SFE_Connectors:1X04_NO_SILK, F.Cu at (131.4, 68.6)
- added J2: Output, SFE_Connectors:1X04_NO_SILK, F.Cu at (166.0, 137.9)
- added J2: Output, SFE_Connectors:1X04_NO_SILK, F.Cu at (96.9, 68.6)
- added J2: Output, SFE_Connectors:1X04_NO_SILK, F.Cu at (131.4, 137.9)
- added J2: Output, SFE_Connectors:1X04_NO_SILK, F.Cu at (96.9, 137.9)
- added J2: Output, SFE_Connectors:1X04_NO_SILK, F.Cu at (200.5, 137.9)
- added J2: Output, SFE_Connectors:1X04_NO_SILK, F.Cu at (235.1, 114.8)
- added J2: Output, SFE_Connectors:1X04_NO_SILK, F.Cu at (166.0, 114.8)
- added J2: Output, SFE_Connectors:1X04_NO_SILK, F.Cu at (131.4, 114.8)
- added J2: Output, SFE_Connectors:1X04_NO_SILK, F.Cu at (96.9, 114.8)
- added LOGO1: SFE_LOGO_NAME_FLAME.1_INCH, SparkFun:SFE_LOGO_NAME_FLAME_.1, B.Cu at (190.0, 133.2)
- added LOGO1: SFE_LOGO_NAME_FLAME.1_INCH, SparkFun:SFE_LOGO_NAME_FLAME_.1, B.Cu at (86.4, 110.1)
- added LOGO1: SFE_LOGO_NAME_FLAME.1_INCH, SparkFun:SFE_LOGO_NAME_FLAME_.1, B.Cu at (190.0, 87.0)
- added LOGO1: SFE_LOGO_NAME_FLAME.1_INCH, SparkFun:SFE_LOGO_NAME_FLAME_.1, B.Cu at (155.4, 87.0)
- added LOGO1: SFE_LOGO_NAME_FLAME.1_INCH, SparkFun:SFE_LOGO_NAME_FLAME_.1, B.Cu at (224.5, 87.0)
- added LOGO1: SFE_LOGO_NAME_FLAME.1_INCH, SparkFun:SFE_LOGO_NAME_FLAME_.1, B.Cu at (120.9, 87.0)
- added LOGO1: SFE_LOGO_NAME_FLAME.1_INCH, SparkFun:SFE_LOGO_NAME_FLAME_.1, B.Cu at (86.4, 87.0)
- added LOGO1: SFE_LOGO_NAME_FLAME.1_INCH, SparkFun:SFE_LOGO_NAME_FLAME_.1, B.Cu at (224.5, 63.9)
- added LOGO1: SFE_LOGO_NAME_FLAME.1_INCH, SparkFun:SFE_LOGO_NAME_FLAME_.1, B.Cu at (190.0, 63.9)
- added LOGO1: SFE_LOGO_NAME_FLAME.1_INCH, SparkFun:SFE_LOGO_NAME_FLAME_.1, B.Cu at (155.4, 63.9)
- added LOGO1: SFE_LOGO_NAME_FLAME.1_INCH, SparkFun:SFE_LOGO_NAME_FLAME_.1, B.Cu at (120.9, 63.9)
- added LOGO1: SFE_LOGO_NAME_FLAME.1_INCH, SparkFun:SFE_LOGO_NAME_FLAME_.1, B.Cu at (155.4, 133.2)
- added LOGO1: SFE_LOGO_NAME_FLAME.1_INCH, SparkFun:SFE_LOGO_NAME_FLAME_.1, B.Cu at (86.4, 63.9)
- added LOGO1: SFE_LOGO_NAME_FLAME.1_INCH, SparkFun:SFE_LOGO_NAME_FLAME_.1, B.Cu at (224.5, 133.2)
- added LOGO1: SFE_LOGO_NAME_FLAME.1_INCH, SparkFun:SFE_LOGO_NAME_FLAME_.1, B.Cu at (120.9, 133.2)
- added LOGO1: SFE_LOGO_NAME_FLAME.1_INCH, SparkFun:SFE_LOGO_NAME_FLAME_.1, B.Cu at (86.4, 133.2)
- added LOGO1: SFE_LOGO_NAME_FLAME.1_INCH, SparkFun:SFE_LOGO_NAME_FLAME_.1, B.Cu at (190.0, 110.1)
- added LOGO1: SFE_LOGO_NAME_FLAME.1_INCH, SparkFun:SFE_LOGO_NAME_FLAME_.1, B.Cu at (155.4, 110.1)
- added LOGO1: SFE_LOGO_NAME_FLAME.1_INCH, SparkFun:SFE_LOGO_NAME_FLAME_.1, B.Cu at (224.5, 110.1)
- added LOGO1: SFE_LOGO_NAME_FLAME.1_INCH, SparkFun:SFE_LOGO_NAME_FLAME_.1, B.Cu at (120.9, 110.1)
- added LOGO2: OSHW-LOGOMINI, Aesthetics:OSHW-LOGO-M, F.Cu at (205.0, 141.7)
- added LOGO2: OSHW-LOGOMINI, Aesthetics:OSHW-LOGO-M, F.Cu at (66.8, 118.5)
- added LOGO2: OSHW-LOGOMINI, Aesthetics:OSHW-LOGO-M, F.Cu at (205.0, 95.4)
- added LOGO2: OSHW-LOGOMINI, Aesthetics:OSHW-LOGO-M, F.Cu at (170.4, 95.4)
- added LOGO2: OSHW-LOGOMINI, Aesthetics:OSHW-LOGO-M, F.Cu at (135.9, 95.4)
- added LOGO2: OSHW-LOGOMINI, Aesthetics:OSHW-LOGO-M, F.Cu at (101.3, 95.4)
- added LOGO2: OSHW-LOGOMINI, Aesthetics:OSHW-LOGO-M, F.Cu at (66.8, 95.4)
- added LOGO2: OSHW-LOGOMINI, Aesthetics:OSHW-LOGO-M, F.Cu at (205.0, 72.3)
- added LOGO2: OSHW-LOGOMINI, Aesthetics:OSHW-LOGO-M, F.Cu at (170.4, 72.3)
- added LOGO2: OSHW-LOGOMINI, Aesthetics:OSHW-LOGO-M, F.Cu at (135.9, 72.3)
- added LOGO2: OSHW-LOGOMINI, Aesthetics:OSHW-LOGO-M, F.Cu at (101.3, 72.3)
- added LOGO2: OSHW-LOGOMINI, Aesthetics:OSHW-LOGO-M, F.Cu at (170.4, 141.7)
- added LOGO2: OSHW-LOGOMINI, Aesthetics:OSHW-LOGO-M, F.Cu at (66.8, 72.3)
- added LOGO2: OSHW-LOGOMINI, Aesthetics:OSHW-LOGO-M, F.Cu at (135.9, 141.7)
- added LOGO2: OSHW-LOGOMINI, Aesthetics:OSHW-LOGO-M, F.Cu at (101.3, 141.7)
- added LOGO2: OSHW-LOGOMINI, Aesthetics:OSHW-LOGO-M, F.Cu at (66.8, 141.7)
- added LOGO2: OSHW-LOGOMINI, Aesthetics:OSHW-LOGO-M, F.Cu at (205.0, 118.5)
- added LOGO2: OSHW-LOGOMINI, Aesthetics:OSHW-LOGO-M, F.Cu at (170.4, 118.5)
- added LOGO2: OSHW-LOGOMINI, Aesthetics:OSHW-LOGO-M, F.Cu at (135.9, 118.5)
- added LOGO2: OSHW-LOGOMINI, Aesthetics:OSHW-LOGO-M, F.Cu at (101.3, 118.5)
- added LOGO3: SFE_LOGO_FLAME.4_INCH, Aesthetics:SFE_LOGO_FLAME_.2, F.Cu at (231.2, 129.3)
- added LOGO3: SFE_LOGO_FLAME.4_INCH, Aesthetics:SFE_LOGO_FLAME_.2, F.Cu at (196.6, 106.2)
- added LOGO3: SFE_LOGO_FLAME.4_INCH, Aesthetics:SFE_LOGO_FLAME_.2, F.Cu at (231.2, 83.1)
- added LOGO3: SFE_LOGO_FLAME.4_INCH, Aesthetics:SFE_LOGO_FLAME_.2, F.Cu at (162.1, 83.1)
- added LOGO3: SFE_LOGO_FLAME.4_INCH, Aesthetics:SFE_LOGO_FLAME_.2, F.Cu at (127.5, 83.1)
- added LOGO3: SFE_LOGO_FLAME.4_INCH, Aesthetics:SFE_LOGO_FLAME_.2, F.Cu at (93.0, 83.1)
- added LOGO3: SFE_LOGO_FLAME.4_INCH, Aesthetics:SFE_LOGO_FLAME_.2, F.Cu at (196.6, 83.1)
- added LOGO3: SFE_LOGO_FLAME.4_INCH, Aesthetics:SFE_LOGO_FLAME_.2, F.Cu at (231.2, 59.9)
- added LOGO3: SFE_LOGO_FLAME.4_INCH, Aesthetics:SFE_LOGO_FLAME_.2, F.Cu at (196.6, 59.9)
- added LOGO3: SFE_LOGO_FLAME.4_INCH, Aesthetics:SFE_LOGO_FLAME_.2, F.Cu at (162.1, 59.9)
- added LOGO3: SFE_LOGO_FLAME.4_INCH, Aesthetics:SFE_LOGO_FLAME_.2, F.Cu at (127.5, 59.9)
- added LOGO3: SFE_LOGO_FLAME.4_INCH, Aesthetics:SFE_LOGO_FLAME_.2, F.Cu at (162.1, 129.3)
- added LOGO3: SFE_LOGO_FLAME.4_INCH, Aesthetics:SFE_LOGO_FLAME_.2, F.Cu at (93.0, 59.9)
- added LOGO3: SFE_LOGO_FLAME.4_INCH, Aesthetics:SFE_LOGO_FLAME_.2, F.Cu at (127.5, 129.3)
- added LOGO3: SFE_LOGO_FLAME.4_INCH, Aesthetics:SFE_LOGO_FLAME_.2, F.Cu at (93.0, 129.3)
- added LOGO3: SFE_LOGO_FLAME.4_INCH, Aesthetics:SFE_LOGO_FLAME_.2, F.Cu at (196.6, 129.3)
- added LOGO3: SFE_LOGO_FLAME.4_INCH, Aesthetics:SFE_LOGO_FLAME_.2, F.Cu at (231.2, 106.2)
- added LOGO3: SFE_LOGO_FLAME.4_INCH, Aesthetics:SFE_LOGO_FLAME_.2, F.Cu at (162.1, 106.2)
- added LOGO3: SFE_LOGO_FLAME.4_INCH, Aesthetics:SFE_LOGO_FLAME_.2, F.Cu at (127.5, 106.2)
- added LOGO3: SFE_LOGO_FLAME.4_INCH, Aesthetics:SFE_LOGO_FLAME_.2, F.Cu at (93.0, 106.2)
- added Ref**: Val**, Pete:STAND-OFF_115_2, F.Cu at (199.0, 142.7)
- added Ref**: Val**, Pete:STAND-OFF_115_2, F.Cu at (66.7, 125.5)
- added Ref**: Val**, Pete:STAND-OFF_115_2, F.Cu at (199.0, 119.6)
- added Ref**: Val**, Pete:STAND-OFF_115_2, F.Cu at (204.9, 102.4)
- added Ref**: Val**, Pete:STAND-OFF_115_2, F.Cu at (233.6, 119.6)
- added Ref**: Val**, Pete:STAND-OFF_115_2, F.Cu at (164.5, 119.6)
- added Ref**: Val**, Pete:STAND-OFF_115_2, F.Cu at (170.3, 102.4)
- added Ref**: Val**, Pete:STAND-OFF_115_2, F.Cu at (135.8, 102.4)
- added Ref**: Val**, Pete:STAND-OFF_115_2, F.Cu at (129.9, 119.6)
- added Ref**: Val**, Pete:STAND-OFF_115_2, F.Cu at (101.2, 102.4)
- added Ref**: Val**, Pete:STAND-OFF_115_2, F.Cu at (95.4, 119.6)
- added Ref**: Val**, Pete:STAND-OFF_115_2, F.Cu at (204.9, 125.5)
- added Ref**: Val**, Pete:STAND-OFF_115_2, F.Cu at (66.7, 102.4)
- added Ref**: Val**, Pete:STAND-OFF_115_2, F.Cu at (199.0, 96.5)
- added Ref**: Val**, Pete:STAND-OFF_115_2, F.Cu at (204.9, 79.2)
- added Ref**: Val**, Pete:STAND-OFF_115_2, F.Cu at (233.6, 96.5)
- added Ref**: Val**, Pete:STAND-OFF_115_2, F.Cu at (164.5, 96.5)
- added Ref**: Val**, Pete:STAND-OFF_115_2, F.Cu at (170.3, 79.2)
- added Ref**: Val**, Pete:STAND-OFF_115_2, F.Cu at (135.8, 79.2)
- added Ref**: Val**, Pete:STAND-OFF_115_2, F.Cu at (129.9, 96.5)
- added Ref**: Val**, Pete:STAND-OFF_115_2, F.Cu at (101.2, 79.2)
- added Ref**: Val**, Pete:STAND-OFF_115_2, F.Cu at (95.4, 96.5)
- added Ref**: Val**, Pete:STAND-OFF_115_2, F.Cu at (233.6, 142.7)
- added Ref**: Val**, Pete:STAND-OFF_115_2, F.Cu at (66.7, 79.2)
- added Ref**: Val**, Pete:STAND-OFF_115_2, F.Cu at (233.6, 73.4)
- added Ref**: Val**, Pete:STAND-OFF_115_2, F.Cu at (204.9, 56.1)
- added Ref**: Val**, Pete:STAND-OFF_115_2, F.Cu at (199.0, 73.4)
- added Ref**: Val**, Pete:STAND-OFF_115_2, F.Cu at (170.3, 56.1)
- added Ref**: Val**, Pete:STAND-OFF_115_2, F.Cu at (164.5, 73.4)
- added Ref**: Val**, Pete:STAND-OFF_115_2, F.Cu at (135.8, 56.1)
- added Ref**: Val**, Pete:STAND-OFF_115_2, F.Cu at (129.9, 73.4)
- added Ref**: Val**, Pete:STAND-OFF_115_2, F.Cu at (101.2, 56.1)
- added Ref**: Val**, Pete:STAND-OFF_115_2, F.Cu at (95.4, 73.4)
- added Ref**: Val**, Pete:STAND-OFF_115_2, F.Cu at (164.5, 142.7)
- added Ref**: Val**, Pete:STAND-OFF_115_2, F.Cu at (66.7, 56.1)
- added Ref**: Val**, Pete:STAND-OFF_115_2, F.Cu at (170.3, 125.5)
- added Ref**: Val**, Pete:STAND-OFF_115_2, F.Cu at (135.8, 125.5)
- added Ref**: Val**, Pete:STAND-OFF_115_2, F.Cu at (129.9, 142.7)
- added Ref**: Val**, Pete:STAND-OFF_115_2, F.Cu at (101.2, 125.5)
- added Ref**: Val**, Pete:STAND-OFF_115_2, F.Cu at (95.4, 142.7)
- added U1: APA102, Pete:APA102_3, F.Cu at (211.6, 140.5)
- added U1: APA102, Pete:APA102_3, F.Cu at (73.4, 117.3)
- added U1: APA102, Pete:APA102_3, F.Cu at (211.6, 94.2)
- added U1: APA102, Pete:APA102_3, F.Cu at (142.5, 94.2)
- added U1: APA102, Pete:APA102_3, F.Cu at (108.0, 94.2)
- added U1: APA102, Pete:APA102_3, F.Cu at (177.0, 94.2)
- added U1: APA102, Pete:APA102_3, F.Cu at (73.4, 94.2)
- added U1: APA102, Pete:APA102_3, F.Cu at (211.6, 71.1)
- added U1: APA102, Pete:APA102_3, F.Cu at (177.0, 71.1)
- added U1: APA102, Pete:APA102_3, F.Cu at (142.5, 71.1)
- added U1: APA102, Pete:APA102_3, F.Cu at (108.0, 71.1)
- added U1: APA102, Pete:APA102_3, F.Cu at (142.5, 140.5)
- added U1: APA102, Pete:APA102_3, F.Cu at (73.4, 71.1)
- added U1: APA102, Pete:APA102_3, F.Cu at (108.0, 140.5)
- added U1: APA102, Pete:APA102_3, F.Cu at (177.0, 140.5)
- added U1: APA102, Pete:APA102_3, F.Cu at (73.4, 140.5)
- added U1: APA102, Pete:APA102_3, F.Cu at (211.6, 117.3)
- added U1: APA102, Pete:APA102_3, F.Cu at (142.5, 117.3)
- added U1: APA102, Pete:APA102_3, F.Cu at (108.0, 117.3)
- added U1: APA102, Pete:APA102_3, F.Cu at (177.0, 117.3)
- added U2: APA102, Pete:APA102_3, F.Cu at (219.2, 140.5)
- added U2: APA102, Pete:APA102_3, F.Cu at (81.0, 117.3)
- added U2: APA102, Pete:APA102_3, F.Cu at (219.2, 94.2)
- added U2: APA102, Pete:APA102_3, F.Cu at (150.1, 94.2)
- added U2: APA102, Pete:APA102_3, F.Cu at (115.6, 94.2)
- added U2: APA102, Pete:APA102_3, F.Cu at (184.7, 94.2)
- added U2: APA102, Pete:APA102_3, F.Cu at (81.0, 94.2)
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Other:
- outline, holes or cut-outs redrawn
