File: Hardware/Lumenati_3x3.kicad_pcb (KiCad board)
At the start: 2 copper layers, 34.3 x 22.9 mm, 25 parts, among them J1 Input, J2 Output, U1 APA102, U2 APA102, U3 APA102, U4 APA102, U5 APA102, U6 APA102, U7 APA102, U8 APA102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

Commit message: Changed silk and file names to Lumenati
Parts:
- moved C1 30.1 mm to (107.4, 95.7)
- moved C3 30.1 mm to (122.7, 95.7)
- moved C4 30.1 mm to (122.7, 81.7)
- moved LOGO1 30.1 mm to (120.4, 85.0)
- moved LOGO2 30.1 mm to (100.8, 93.4)
- moved C6 30.1 mm to (107.4, 81.7)
- moved U1 30.1 mm to (107.4, 92.2)
- moved U2 30.1 mm to (115.1, 92.2)
- moved U3 30.1 mm to (122.7, 92.2)
- moved U4 30.1 mm to (122.7, 85.2)
- moved U5 30.1 mm to (115.1, 85.2)
- moved U6 30.1 mm to (107.4, 85.2)
- moved U7 30.1 mm to (107.4, 78.2)
- moved U8 30.1 mm to (115.1, 78.2)
- moved U9 30.1 mm to (122.7, 78.2)
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Other:
- board text added: "Lumenati 3x3"
- board text added: "v10"
- board text removed: "HiBeam 3x3"
- board text removed: "HiBeams 3x3"
- board text removed: "v01"
