File: Hardware/Lumenati_3x3.sch (KiCad schematic (older format))
At the start: 22 parts, among them J1 Input, J2 Output, U1 APA102, U2 APA102, U3 APA102, U4 APA102, U5 APA102, U6 APA102, U7 APA102, U8 APA102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

Commit message: Changed silk and file names to Lumenati
Other:
- note added: "Lumenati 3x3"
- note added: "v10"
- note removed: "HiBeams 3x3"
- note removed: "v01"
Changed lines of the file:
@@
 LIBS:contrib
 LIBS:valves
-LIBS:apa102c
-LIBS:LilyPad-Wearables
-LIBS:SparkFun-Aesthetics
-LIBS:SparkFun-Batteries
-LIBS:SparkFun-Boards
-LIBS:SparkFun-Capacitors
-LIBS:SparkFun-Clocks
-LIBS:SparkFun-Coils
-LIBS:SparkFun-Connectors
-LIBS:SparkFun-DiscreteSemi
-LIBS:SparkFun-Displays
-LIBS:SparkFun-Electromechanical
-LIBS:SparkFun-Fuses
-LIBS:SparkFun-GPS
-LIBS:SparkFun-Hardware
-LIBS:SparkFun-IC-Amplifiers
-LIBS:SparkFun-IC-Comms
-LIBS:SparkFun-IC-Conversion
-LIBS:SparkFun-IC-Logic
-LIBS:SparkFun-IC-Memory
-LIBS:SparkFun-IC-Microcontroller
-LIBS:SparkFun-IC-Power
-LIBS:SparkFun-IC-Special-Function
-LIBS:SparkFun-Jumpers
-LIBS:SparkFun-LED
-LIBS:SparkFun-PowerSymbols
-LIBS:SparkFun-Resistors
-LIBS:SparkFun-RF
-LIBS:SparkFun-Sensors
-LIBS:SparkFun-Switches
-LIBS:Hi-beam quad-cache
-LIBS:APA102
 LIBS:HiBeam_3x3-cache
-EELAYER 26 0
+EELAYER 25 0
 EELAYER END
 $Descr A4 11693 8268
@@
 $EndComp
 Text Notes 10600 7650 0    60   ~ 0
-v01
+v10
 Text Notes 8250 7650 0    60   ~ 0
 6/1/17
 Text Notes 7350 7500 0    60   ~ 0
-HiBeams 3x3
+Lumenati 3x3
 $Comp
 L +5V #PWR07
